Commit message: C011 connection, works

File: structure_synthesis/kinematic_verification_011.xacro (robot description, xacro)
@@ -9,13 +9,13 @@
 <xacro:property name="final_theta_p_1" value="${0+theta_p_1}"/>
 <xacro:property name="theta_p_2" value="0"/>
-<xacro:property name="final_theta_p_2" value="${3.1416+theta_p_2}"/>
-<!-- Synthetic C01-->
-<xacro:property name="Rx01" value="0"/>
-<xacro:property name="Ry01" value="0"/>
-<xacro:property name="Rz01" value="0"/>
-<xacro:property name="Px01" value="0"/>
-<xacro:property name="fPx01" value="${0.091+Px01}"/>
-<xacro:property name="Py01" value="0"/>
-<xacro:property name="Pz01" value="0"/>
+<xacro:property name="final_theta_p_2" value="${0+theta_p_2}"/>
+<!-- Synthetic C011-->
+<xacro:property name="Rx011" value="1.5708"/>
+<xacro:property name="Ry011" value="0"/>
+<xacro:property name="Rz011" value="0"/>
+<xacro:property name="Px011" value="0"/>
+<xacro:property name="fPx011" value="${0.091+Px011}"/>
+<xacro:property name="Py011" value="0.05"/>
+<xacro:property name="Pz011" value="0.05"/>
 <!-- Synthetic C10 is always to zero, just in case Vassilis orders-->
 <xacro:property name="Rx10" value="0"/>
@@ -101,5 +101,5 @@
 <!-- This joint is parameterized for C01-->
   <joint name="frame__PseudoConnector1a" type="fixed">
-    <origin rpy="${Rx01} ${Ry01} ${Rz01}" xyz="${fPx01} ${Py01} ${Pz01}"/>
+    <origin rpy="${Rx011} ${Ry011} ${Rz011}" xyz="${fPx011} ${Py011} ${Pz011}"/>
     <parent link="frame"/>
     <child link="PseudoConnector1a"/>
@@ -147,5 +147,5 @@
 <!-- END of pseudojoint1 -->
   <joint name="PseudoConnector1b__PseudoConnector2a" type="fixed">
-    <origin rpy="0 0 1.5708" xyz="0 0 0.032"/>
+    <origin rpy="0 0 -1.5708" xyz="0 0 0.032"/>
     <parent link="PseudoConnector1b"/>
     <child link="PseudoConnector2a"/>
@@ -182,5 +182,5 @@
     </inertial>
     <visual>
-      <origin rpy="0 0 0" xyz="0 -0.010 -0.027"/>
+      <origin rpy="0 3.1416 0" xyz="0 -0.010 0.027"/>
       <geometry>
         <mesh filename="/home/nikos/matlab_ws/modular_dynamixel/pseudo.stl" scale="0.001 0.001 0.001"/>
@@ -193,5 +193,5 @@
 <!-- END of pseudojoint2 -->
   <joint name="PseudoConnector2b__adaptor1" type="fixed">
-    <origin rpy="0 3.14 -1.57" xyz="0 -0.010 -0.032"/>
+    <origin rpy="0 0 1.57" xyz="0 -0.010 0.032"/>
     <parent link="PseudoConnector2b"/>
     <child link="adaptor1"/>

Commit message: changes to counterbalance lost files

File: structure_synthesis/kinematic_verification_011.xacro (robot description, xacro)
@@ -37,12 +37,12 @@
 <link name="base_link">
     <inertial>
-      <origin rpy="0 0 0" xyz="0.0021 -0.0033 -0.00574"/>
-      <mass value ="0.855" />
-      <inertia ixx="0.0040487283" ixy="0.000016444686" ixz="0.0001418628" iyy="0.0040350489" iyz="-0.0002178358" izz="0.0003489357"/>
+      <origin rpy="0 0 0" xyz="0.00205 0.00373 0.020774"/>
+      <mass value ="0.675" />
+      <inertia ixx="5.063e-004" ixy="2.773e-005" ixz="7.042e-007" iyy="5.387e-004" iyz="1.237e-006" izz="7.207e-004"/>
     </inertial>
     <visual>
       <origin rpy="1.57 0 0" xyz="0 0 0.120"/>
       <geometry>
-        <mesh filename="/home/nikos/matlab_ws/modular_dynamixel/H54P-200.stl" scale="0.001 0.001 0.001"/>
+        <mesh filename="/home/nikos/PhD/projects/Dynamics_SMM/baselink/ovidius_smm_baselink.stl" scale="0.001 0.001 0.001"/>
       </geometry>
       <material name="gray">
@@ -52,10 +52,10 @@
 </link>
 <!-- START ONLY visual representation of adaptor to lock base in table-->
-  <joint name="base_link__adaptor" type="fixed">
+  <joint name="base_link__pseudo1a" type="fixed">
     <origin rpy="0 0 0" xyz="-0.030 0 0.057"/>
     <parent link="base_link"/>
     <child link="adaptor"/>
   </joint>
-<link name="adaptor">
+<link name="pseudo1a">
       <inertial>
         <origin rpy="0 0 0" xyz="0 0.00132 0"/>
